File: Electrical/Design/EN16/EN16/EN16.sch (KiCad schematic (older format))
At the start: 0 parts

Commit message: SUKU EN16 PCB routing finished
Connections:
- no-connect marks 1 -> 6
Changed lines of the file:
@@
 F9 "HWCFG_CLOCK" O R 11000 6600 50
 F10 "HWCFG_SHIFT" O R 11000 6500 50
+F11 "UI_SPI_MOSI" O L 9000 5100 50
+F12 "UI_SPI_MISO" I L 9000 5200 50
+F13 "UI_SPI_SCK" O L 9000 5300 50
+F14 "UI_SPI_CS" O L 9000 5400 50
 $EndSheet
 Wire Wire Line
@@
 F0 "UI_ENC" 50
 F1 "UI_ENC.sch" 50
+F2 "ENCODER_MISO" O R 8000 5200 50
+F3 "ENCODER_MOSI" I R 8000 5100 50
+F4 "ENCODER_SCK" I R 8000 5300 50
+F5 "ENCODER_CS" I R 8000 5400 50
 $EndSheet
+Wire Wire Line
+	8000 5100 9000 5100
+Wire Wire Line
+	9000 5200 8000 5200
+Wire Wire Line
+	8000 5300 9000 5300
+Wire Wire Line
+	9000 5400 8000 5400
+Wire Wire Line
+	9000 6400 8800 6400
+Wire Wire Line
+	9000 6500 8800 6500
+Wire Wire Line
+	9000 6700 8800 6700
+Wire Wire Line
+	9000 6800 8800 6800
+Wire Wire Line
+	9000 6900 8800 6900
+NoConn ~ 8800 6400
+NoConn ~ 8800 6500
+NoConn ~ 8800 6700
+NoConn ~ 8800 6800
+NoConn ~ 8800 6900
 $EndSCHEMATC
