File: Electrical/Design/PO16_BU16/PO16_BU16/UI_LED.sch (KiCad schematic (older format))
At the start: 32 parts

Commit message: SUKU POBU16 PBF4 sync progress
Connections:
- net +3V3_UI renamed +5V_UI
