File: Electrical/Design/TEK2/TEK2/TEK2.kicad_sch (KiCad schematic)
At the start: 0 parts

Commit message: SUKU TEK2 sch and layout done
Other:
- sheet UI_BUTTON ports: added none; removed OUT_0, OUT_1, OUT_2, OUT_3, OUT_4, OUT_5, OUT_6, OUT_7
- sheet UI_POT ports: added none; removed OUT_10, OUT_11, OUT_12, OUT_13, OUT_14, OUT_15, OUT_8, OUT_9
Changed lines of the file:
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@@
-    (stroke (width 0) (type default))
-  )
-  (wire (pts (xy 132.08 172.72) (xy 127 172.72))
     (stroke (width 0) (type default))
   )
@@
     (stroke (width 0) (type default))
   )
-  (wire (pts (xy 127 142.24) (xy 132.08 142.24))
-    (stroke (width 0) (type default))
-  )
   (wire (pts (xy 228.6 104.14) (xy 203.2 104.14))
     (stroke (width 0) (type default))
   )
-  (wire (pts (xy 127 175.26) (xy 132.08 175.26))
-    (stroke (width 0) (type default))
-  )
   (wire (pts (xy 175.26 198.12) (xy 170.18 198.12))
     (stroke (width 0) (type default))
@@
     (stroke (width 0) (type default))
   )
-  (wire (pts (xy 127 160.02) (xy 132.08 160.02))
-    (stroke (width 0) (type default))
-  )
   (wire (pts (xy 132.08 190.5) (xy 127 190.5))
     (stroke (width 0) (type default))
@@
     (stroke (width 0) (type default))
   )
-  (wire (pts (xy 132.08 129.54) (xy 127 129.54))
-    (stroke (width 0) (type default))
-  )
-  (wire (pts (xy 132.08 144.78) (xy 127 144.78))
-    (stroke (width 0) (type default))
-  )
   (wire (pts (xy 132.08 195.58) (xy 127 195.58))
     (stroke (width 0) (type default))
@@
     (stroke (width 0) (type default))
   )
-  (wire (pts (xy 127 157.48) (xy 132.08 157.48))
-    (stroke (width 0) (type default))
-  )
   (wire (pts (xy 200.66 200.66) (xy 215.9 200.66))
     (stroke (width 0) (type default))
@@
     (stroke (width 0) (type default))
   )
-  (wire (pts (xy 127 147.32) (xy 132.08 147.32))
-    (stroke (width 0) (type default))
-  )
   (wire (pts (xy 175.26 187.96) (xy 170.18 187.96))
     (stroke (width 0) (type default))
@@
     (stroke (width 0) (type default))
   )
-  (wire (pts (xy 127 165.1) (xy 132.08 165.1))
-    (stroke (width 0) (type default))
-  )
   (wire (pts (xy 279.4 167.64) (xy 304.8 167.64))
     (stroke (width 0) (type default))
@@
     (stroke (width 0) (type default))
   )
-  (wire (pts (xy 127 170.18) (xy 132.08 170.18))
-    (stroke (width 0) (type default))
-  )
-  (wire (pts (xy 132.08 167.64) (xy 127 167.64))
-    (stroke (width 0) (type default))
-  )
-  (wire (pts (xy 132.08 139.7) (xy 127 139.7))
-    (stroke (width 0) (type default))
-  )
   (wire (pts (xy 200.66 198.12) (xy 215.9 198.12))
     (stroke (width 0) (type default))
   )
-  (wire (pts (xy 132.08 134.62) (xy 127 134.62))
-    (stroke (width 0) (type default))
-  )
   (wire (pts (xy 127 193.04) (xy 132.08 193.04))
     (stroke (width 0) (type default))
@@
     (stroke (width 0) (type default))
   )
-  (wire (pts (xy 127 132.08) (xy 132.08 132.08))
-    (stroke (width 0) (type default))
-  )
-  (wire (pts (xy 132.08 162.56) (xy 127 162.56))
-    (stroke (width 0) (type default))
-  )
   (wire (pts (xy 175.26 231.14) (xy 170.18 231.14))
-    (stroke (width 0) (type default))
-  )
-  (wire (pts (xy 127 137.16) (xy 132.08 137.16))
     (stroke (width 0) (type default))
   )
@@
     (effects (font (size 1.27 1.27)) (justify right bottom))
   )
-  (label "ANA_6" (at 132.08 172.72 0) (fields_autoplaced)
-    (effects (font (size 1.27 1.27)) (justify left bottom))
-  )
   (label "ANA_8" (at 132.08 185.42 0) (fields_autoplaced)
     (effects (font (size 1.27 1.27)) (justify left bottom))
@@
     (effects (font (size 1.27 1.27)) (justify right bottom))
   )
-  (label "ANA_2" (at 132.08 162.56 0) (fields_autoplaced)
-    (effects (font (size 1.27 1.27)) (justify left bottom))
-  )
-  (label "ANA_11" (at 132.08 137.16 0) (fields_autoplaced)
-    (effects (font (size 1.27 1.27)) (justify left bottom))
-  )
-  (label "ANA_9" (at 132.08 132.08 0) (fields_autoplaced)
-    (effects (font (size 1.27 1.27)) (justify left bottom))
-  )
-  (label "ANA_5" (at 132.08 170.18 0) (fields_autoplaced)
-    (effects (font (size 1.27 1.27)) (justify left bottom))
-  )
-  (label "ANA_3" (at 132.08 165.1 0) (fields_autoplaced)
-    (effects (font (size 1.27 1.27)) (justify left bottom))
-  )
   (label "ANA_7" (at 170.18 223.52 180) (fields_autoplaced)
     (effects (font (size 1.27 1.27)) (justify right bottom))
   )
-  (label "ANA_7" (at 132.08 175.26 0) (fields_autoplaced)
-    (effects (font (size 1.27 1.27)) (justify left bottom))
-  )
-  (label "ANA_4" (at 132.08 167.64 0) (fields_autoplaced)
-    (effects (font (size 1.27 1.27)) (justify left bottom))
-  )
   (label "ANA_2" (at 170.18 215.9 180) (fields_autoplaced)
     (effects (font (size 1.27 1.27)) (justify right bottom))
   )
-  (label "ANA_0" (at 132.08 157.48 0) (fields_autoplaced)
-    (effects (font (size 1.27 1.27)) (justify left bottom))
-  )
-  (label "ANA_1" (at 132.08 160.02 0) (fields_autoplaced)
-    (effects (font (size 1.27 1.27)) (justify left bottom))
-  )
   (label "ANA_3" (at 132.08 109.22 0) (fields_autoplaced)
     (effects (font (size 1.27 1.27)) (justify left bottom))
   )
-  (label "ANA_14" (at 132.08 144.78 0) (fields_autoplaced)
-    (effects (font (size 1.27 1.27)) (justify left bottom))
-  )
-  (label "ANA_12" (at 132.08 139.7 0) (fields_autoplaced)
-    (effects (font (size 1.27 1.27)) (justify left bottom))
-  )
-  (label "ANA_10" (at 132.08 134.62 0) (fields_autoplaced)
-    (effects (font (size 1.27 1.27)) (justify left bottom))
-  )
   (label "ANA_13" (at 132.08 198.12 0) (fields_autoplaced)
     (effects (font (size 1.27 1.27)) (justify left bottom))
   )
-  (label "ANA_13" (at 132.08 142.24 0) (fields_autoplaced)
-    (effects (font (size 1.27 1.27)) (justify left bottom))
-  )
   (label "ANA_12" (at 170.18 200.66 180) (fields_autoplaced)
     (effects (font (size 1.27 1.27)) (justify right bottom))
@@
     (effects (font (size 1.27 1.27)) (justify right bottom))
   )
-  (label "ANA_8" (at 132.08 129.54 0) (fields_autoplaced)
-    (effects (font (size 1.27 1.27)) (justify left bottom))
-  )
   (label "ANA_0" (at 132.08 101.6 0) (fields_autoplaced)
     (effects (font (size 1.27 1.27)) (justify left bottom))
@@
   (label "ANA_3" (at 170.18 218.44 180) (fields_autoplaced)
     (effects (font (size 1.27 1.27)) (justify right bottom))
-  )
-  (label "ANA_15" (at 132.08 147.32 0) (fields_autoplaced)
-    (effects (font (size 1.27 1.27)) (justify left bottom))
   )
   (label "ANA_14" (at 132.08 200.66 0) (fields_autoplaced)
@@
       (effects (font (size 1.27 1.27)) (justify right))
     )
-    (pin "OUT_8" passive (at 127 129.54 0)
-      (effects (font (size 1.27 1.27)) (justify right))
-    )
-    (pin "OUT_9" passive (at 127 132.08 0)
-      (effects (font (size 1.27 1.27)) (justify right))
-    )
-    (pin "OUT_10" passive (at 127 134.62 0)
-      (effects (font (size 1.27 1.27)) (justify right))
-    )
-    (pin "OUT_11" passive (at 127 137.16 0)
-      (effects (font (size 1.27 1.27)) (justify right))
-    )
-    (pin "OUT_13" passive (at 127 142.24 0)
-      (effects (font (size 1.27 1.27)) (justify right))
-    )
-    (pin "OUT_12" passive (at 127 139.7 0)
-      (effects (font (size 1.27 1.27)) (justify right))
-    )
-    (pin "OUT_14" passive (at 127 144.78 0)
-      (effects (font (size 1.27 1.27)) (justify right))
-    )
-    (pin "OUT_15" passive (at 127 147.32 0)
-      (effects (font (size 1.27 1.27)) (justify right))
-    )
     (instances
       (project "TEK2"
@@
       (effects (font (size 1.27 1.27)) (justify right))
     )
-    (pin "OUT_3" passive (at 127 165.1 0)
-      (effects (font (size 1.27 1.27)) (justify right))
-    )
-    (pin "OUT_2" passive (at 127 162.56 0)
-      (effects (font (size 1.27 1.27)) (justify right))
-    )
     (pin "OUT_11" passive (at 127 193.04 0)
       (effects (font (size 1.27 1.27)) (justify right))
@@
       (effects (font (size 1.27 1.27)) (justify right))
     )
-    (pin "OUT_7" passive (at 127 175.26 0)
-      (effects (font (size 1.27 1.27)) (justify right))
-    )
-    (pin "OUT_6" passive (at 127 172.72 0)
-      (effects (font (size 1.27 1.27)) (justify right))
-    )
-    (pin "OUT_1" passive (at 127 160.02 0)
-      (effects (font (size 1.27 1.27)) (justify right))
-    )
-    (pin "OUT_5" passive (at 127 170.18 0)
-      (effects (font (size 1.27 1.27)) (justify right))
-    )
-    (pin "OUT_4" passive (at 127 167.64 0)
-      (effects (font (size 1.27 1.27)) (justify right))
-    )
-    (pin "OUT_0" passive (at 127 157.48 0)
-      (effects (font (size 1.27 1.27)) (justify right))
-    )
