File: Electrical/Design/PCBA-XX16-FRONTPANEL/PCBA-XX16-FRONTPANEL.kicad_sch (KiCad schematic)
At the start: 0 parts

Commit message: SUKU all pcb frontpanels updated to use proper footprints, silkscreen variables and design rules
Parts:
- added H501, H503, H505, H507, H509, H511, H513, H515, H517, H519, H521, H523, H525, H527, H529, H531: LED, suku_basics:FP_LED, symbol Mechanical:MountingHole
- added H502, H504, H506, H508, H510, H512, H514, H516, H518, H520, H522, H524, H526, H528, H530, H532: Potentiometer, suku_basics:FP_POTENTIOMETER, symbol Mechanical:MountingHole
- added H533: Outline, suku_basics:FP_OUTLINE, symbol Mechanical:MountingHole
