File: Electrical/Design/FP-EN16-MIDIGRADE/FP-EN16-MIDIGRADE.kicad_sch (KiCad schematic)
At the start: 34 parts

Commit message: SUKU midigrad test added
Parts:
- H501, H503, H505, H507, H509, H511, H513, H515, H517, H519, H521, H523, H525, H527, H529, H531: footprint suku_basics:FP_LED -> suku_basics:FP_LED_TIGHT; symbol Mechanical:MountingHole -> Mechanical:MountingHole_Pad; now in the parts list
Connections:
- new net GND: H501.1, H503.1, H505.1, H507.1, H509.1, H511.1, H513.1, H515.1, H517.1, H519.1, H521.1, H523.1, H525.1, H527.1, H529.1, H531.1
