File: Electrical/Design/PCBA-OCTV/INVERT_AND_OFFSET.kicad_sch (KiCad schematic)
At the start: 6 parts, among them U1025 LMV321

Commit message: SUKU keyswitch positioning done
Parts:
- removed U1025: LMV321, suku_basics:SOT-23-5, symbol Amplifier_Operational:LM321
- added R624, R654, R656: 10k, suku_basics:RES_0402, symbol suku_basics:RES
- added R625, R655, R657, R720, R721, R722: 15k, suku_basics:RES_0402, symbol suku_basics:RES
- added R687, R688, R689: 5k1, suku_basics:RES_0402, symbol suku_basics:RES
- added U623: LMV324, Package_SO:SOIC-14_3.9x8.7mm_P1.27mm, symbol Amplifier_Operational:LMV324
- renumbered C1041 to C608, R1042 to R622, R1043 to R623, R1041 to R686, R1044 to R719
Connections:
- net INPUT is gone; now on an unnamed net: R686.2
- net +3V3: now also R624.2, R654.2, R656.2, U623.4 (V+)
- net GND: now also R623.2, R625.2, R655.2, R657.2, U623.11 (V-); no longer R623.1
- net at R622.1: now also R623.1, U623.3 (+); no longer R623.2
- net at R719.2: now also U623.2 (-); no longer R686.1
- net OUTPUT renamed OUTPUT_0
- net OUTPUT_0: now also U623.1
- new net: R689.2, R722.2, U623.13 (-)
- new net: R687.2, R720.2, U623.6 (-)
- new net: R654.1, R655.1, U623.10 (+)
- new net: R624.1, R625.1, U623.5 (+)
- new net: R688.2, R721.2, U623.9 (-)
- new net: R656.1, R657.1, U623.12 (+)
- new net INPUT_0: R686.1
- new net INPUT_1: R687.1
- new net INPUT_2: R688.1
- new net INPUT_3: R689.1
- new net OUTPUT_1: R720.1, U623.7
- new net OUTPUT_2: R721.1, U623.8
- new net OUTPUT_3: R722.1, U623.14
Other:
- moved on the sheet: C608, R622, R623, R686, R719
