File: Electrical/Design/PCBA-OCTV/PCBA-OCTV.kicad_pcb (KiCad board)
At the start: 4 copper layers, 100 x 100 mm, 403 parts, among them J1005 SMTSO1625MTJ, J1006 SMTSO1625MTJ, J1007 SMTSO1625MTJ, J1008 SMTSO1625MTJ, J501 Conn_01x04, J502 Conn_01x04, J503 Conn_01x04, J504 Conn_01x04, J505 Conn_01x04, J506 Conn_01x04, J507 Conn_01x04, J508 Conn_01x04, J601 TYPE-C-32-M-12, J602 SMTSO1625MTJ, J603 SMTSO1625MTJ, J604 SMTSO1625MTJ, J605 SMTSO1625MTJ, J701 C5137195, J702 Conn_02x05_Odd_Even, J799 Conn_01x02, M501 Conn_01x08, SW1001 C2905169, SW1002 C2905169, SW1003 C2905169, SW1004 C2905169, SW1005 C2905169, SW1006 C2905169, SW1007 C2905169, SW1008 C2905169, SW1009 C2905169, SW1010 C2905169, SW1011 C2905169, SW1013 C2905169, SW1015 C2905169, SW701 C255807, SW702 C2905169, SW703 C2905169, U1001 74HC4051, U1002 74HC4051, U1003 OH49E-S, U1004 OH49E-S, U1005 OH49E-S, U1006 OH49E-S, U1007 OH49E-S, U1008 OH49E-S, U1009 OH49E-S, U1010 OH49E-S, U1011 OH49E-S, U1012 OH49E-S, U1013 OH49E-S, U1014 74HC165, U1015 OH49E-S, U1016 74HC165, U1017 OH49E-S, U1018 74HC165, U1019 74HC165, U601 LN1134A332MR-G, U602 C5451661, U603 C5451661, U604 74LVC1G08, U605 BL1551B, U606 BL1551B, U607 BL1551B, U608 BL1551B, U609 LMV321, U610 LMV321, U611 LMV321, U612 LMV321, U613 LMV321, U614 LMV321, U615 LMV321, U616 LMV321, U617 LMV321, U618 LMV321, U619 LMV321, U620 LMV321, U621 LMV321, U622 LMV321, U623 LMV321, U624 LMV321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

Commit message: SUKU custom grid outline created and added
Parts:
- M501: footprint suku_basics:grid_outline -> suku_basics:grid_outline_octv
- moved M501 236.7 mm to (100.0, 100.0)

Commit message: SUKU HWCFG adjusted, solder bridge selector for smooth varian added, grid port layout added to layout group
Parts:
- added JP1001: (NF), Jumper:SolderJumper-2_P1.3mm_Open_TrianglePad1.0x1.5mm, F.Cu at (105.2, 75.5)
- added R1065: 5k1, suku_basics:RES_0402, F.Cu at (105.2, 73.0)
- moved J1005 256.8 mm to (33.9, 135.9)
- moved J1006 256.8 mm to (33.9, 142.0)
- moved J602 256.8 mm to (21.7, 135.9)
- moved J603 256.8 mm to (21.7, 142.0)
- moved J1007 256.8 mm to (40.0, 135.9)
- moved J1008 256.8 mm to (40.0, 142.0)
- moved J604 256.8 mm to (27.8, 135.9)
- moved J605 256.8 mm to (27.8, 142.0)
Connections:
- U801 pad 12: GND -> +3V3
- U801 pad 14: GND -> +3V3
- U801 pad 3: GND -> Net-(JP1001-B)
Routing:
- net Net-(JP1001-B): track 0.00 -> 6.27 mm, vias 0 -> 1
- net +3V3: track 86.4 -> 92.5 mm, vias 50 -> 53
- net GND: track 202.7 -> 200.9 mm, vias 90 -> 87
- net /MCU/U0TXD: track 78.2 -> 77.0 mm
- net /MCU/ESP_RESET: track 65.8 -> 66.6 mm
Other:
- board text added: "ND"

Commit message: SUKU audio circuit imported brom VSNX
Parts:
- added ?: , , F.Cu at (205.0, 111.2)
- added C1030: 10u, suku_basics:CAP_0402, B.Cu at (206.0, 107.5)
- added C1062: 1u, suku_basics:CAP_0402, B.Cu at (207.0, 107.5)
- added C1063: 100n, suku_basics:CAP_0402, B.Cu at (208.0, 107.5)
- added C1066: 1n, suku_basics:CAP_0402, B.Cu at (209.8, 110.5)
- added C1069: 1n, suku_basics:CAP_0402, B.Cu at (209.8, 111.8)
- added L1001: BLM15PD121SN1D, suku_basics:FERRIT_0402, B.Cu at (204.5, 107.0)
- added L1002: BLM15AG102SN1D, suku_basics:FERRIT_0402, B.Cu at (209.8, 113.0)
- added L1003: BLM15AG102SN1D, suku_basics:FERRIT_0402, B.Cu at (209.8, 109.2)
- added LS1001: Speaker, suku_basics:speaker-1609, B.Cu at (205.0, 131.2)
- added R1066: 0R, suku_basics:RES_0402, B.Cu at (204.5, 108.0)
- added R1067: 33R, suku_basics:RES_0402, B.Cu at (200.0, 111.8)
- added R1068: 33R, suku_basics:RES_0402, B.Cu at (200.0, 110.5)
- added R1069: 33R, suku_basics:RES_0402, B.Cu at (200.0, 109.2)
- added R1070: 33R, suku_basics:RES_0402, B.Cu at (204.0, 121.8)
- added R1071: 33R, suku_basics:RES_0402, B.Cu at (205.0, 121.8)
- added R1072: 33R, suku_basics:RES_0402, B.Cu at (206.0, 121.8)
- added TP1001: TestPoint, TestPoint:TestPoint_Pad_D1.0mm, B.Cu at (211.8, 112.8)
- added TP1002: TestPoint, TestPoint:TestPoint_Pad_D1.0mm, B.Cu at (211.8, 109.8)
- added TP1003: TestPoint, TestPoint:TestPoint_Pad_D1.0mm, B.Cu at (211.8, 111.2)
- added U1020: NS4168_C910588, suku_basics:ESOP-8_L4.9-W3.9-P1.27-LS6.0-BL-EP, B.Cu at (205.0, 111.2)
Connections:
- net /MCU/TCK renamed ESP_GPIO_39
- net /MCU/TDI renamed ESP_GPIO_41
- net /MCU/TDO renamed ESP_GPIO_40
- net /MCU/TMS renamed ESP_GPIO_42
- net /MCU/U0RXD renamed ESP_GPIO_44
- net /MCU/U0TXD renamed ESP_GPIO_43
Routing:
- net Net-(C1066-Pad1): track 0.00 -> 29.8 mm
- net Net-(C1069-Pad1): track 0.00 -> 24.2 mm
- net +3.3VA: track 0.00 -> 17.5 mm
- net GNDA: track 0.00 -> 13.6 mm
- net Net-(U1020-SDATA): track 0.00 -> 1.49 mm
- net Net-(U1020-BCLK): track 0.00 -> 1.47 mm
- net Net-(U1020-LRCLK): track 0.00 -> 1.44 mm
- net Net-(U1020-VOP): track 0.00 -> 1.40 mm
- net Net-(U1020-VON): track 0.00 -> 1.24 mm
- net GND: track 200.9 -> 201.6 mm, vias 87 -> 88
- net +3V3: track 92.5 -> 93.3 mm, vias 53 -> 54
