File: Electrical/Design/PCBA-BU16/INVERT_AND_OFFSET.kicad_sch (KiCad schematic)
At the start: 6 parts, among them U1025 LMV321

Commit message: SUKU sch + layout progress
Parts:
- renumbered C1041 to C1035, R1041 to R1017, R1042 to R1018, R1043 to R1019, R1044 to R1020, U1025 to U1019
Changed lines of the file:
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@@
 (kicad_sch
-	(version 20231120)
+	(version 20250114)
 	(generator "eeschema")
-	(generator_version "8.0")
+	(generator_version "9.0")
 	(paper "A4")
 	(junction
@@
 		(on_board yes)
 		(dnp no)
-		(property "Reference" "R1042"
+		(property "Reference" "R1018"
 			(at 96.4184 66.04 90)
 			(effects
@@
 		(on_board yes)
 		(dnp no)
-		(property "Reference" "R1041"
+		(property "Reference" "R1017"
 			(at 83.82 71.2216 90)
 			(effects
@@
 		(on_board yes)
 		(dnp no)
-		(property "Reference" "U1025"
+		(property "Reference" "U1019"
 			(at 101.6 78.74 0)
 			(effects
@@
 		(on_board yes)
 		(dnp no)
-		(property "Reference" "R1043"
+		(property "Reference" "R1019"
 			(at 96.4184 81.28 90)
 			(effects
@@
 		(dnp no)
 		(fields_autoplaced yes)
-		(property "Reference" "#PWR01131"
+		(property "Reference" "#PWR01107"
 			(at 99.06 95.25 0)
 			(effects
@@
 		(on_board yes)
 		(dnp no)
-		(property "Reference" "C1041"
+		(property "Reference" "C1035"
 			(at 124.2568 57.2516 0)
 			(effects
@@
 		(dnp no)
 		(fields_autoplaced yes)
-		(property "Reference" "#PWR01130"
+		(property "Reference" "#PWR01106"
 			(at 99.06 57.15 0)
 			(effects
@@
 		(on_board yes)
 		(dnp no)
-		(property "Reference" "R1044"
+		(property "Reference" "R1020"
 			(at 104.14 53.4416 90)
 			(effects
@@
 		(dnp no)
 		(fields_autoplaced yes)
-		(property "Reference" "#PWR01133"
+		(property "Reference" "#PWR01109"
 			(at 121.92 69.85 0)
 			(effects
@@
 		(dnp no)
 		(fields_autoplaced yes)
-		(property "Reference" "#PWR01132"
+		(property "Reference" "#PWR01108"
 			(at 121.92 57.15 0)
 			(effects
