File: Electrical/Design/PCBA-BU16/INVERT_AND_OFFSET.kicad_sch (KiCad schematic)
At the start: 6 parts, among them U1019 LMV321

Commit message: SUKU annotation checker added, wired into CI; BU16/EF44 reannotated
check_annotation.py verifies a schematic sheet instance's reference
designators against this repo's actual page-number-driven annotation
strategy (KiCad's "First free after sheet number X 100"), without
invoking KiCad — there's no headless reannotate to diff against, since
kicad-cli has no `sch annotate` and eeschema has no scripting console.
A sheet instance's page number gives it an exclusive numbering block;
each reference prefix gets its own Y-then-X sorted counter within it.
Multiply-instantiated sheets (e.g. UI_ENC_FILTER placed 4x, or
INVERT_AND_OFFSET nested 8x inside each of UI_HALL_PREAMP's 2
placements) are matched and checked per instance via KiCad's own
hierarchical path chains, not per file.

A preflight, required before any per-symbol check, walks the sheet
hierarchy from the project root (following Sheetfile references, same
as KiCad) and enforces two invariants the KiCad GUI does not: every
sheet instance's page number must be globally unique, and page numbers
must be contiguous from 1 with no gaps. It also flags .kicad_sch files
present in a design folder but unreachable from the root as orphans.

Wired into CI as "annotation-check" / "annotation gate", same pattern
as the existing schematic-drift/design-rules gates: GitHub Actions
error annotations plus a job-summary table when GITHUB_ACTIONS=true.
generate-artifacts now depends on it too.

Preflight caught a real bug in BU16: UI_HALL_PREAMP is placed twice,
and both placements' 8 nested INVERT_AND_OFFSET instances had been
assigned the same page numbers (11-18 each, duplicated) instead of
each getting its own range — invisible in KiCad's hierarchy panel
without instance-aware tooling. Fixed by renumbering one branch to
10-17 and the other to 19-26, then reannotating every sheet in both
EF44 and BU16 to match; both now pass with zero mismatches.

Also removed 6 orphaned .kicad_sch files (leftover from EF44's fork
off BU16 replacin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
Parts:
- renumbered C1035 to C1001, R1020 to R1001, R1018 to R1002, R1017 to R1003, R1019 to R1004, U1019 to U1001
