File: Electrical/Design/PCBA-BU16/INVERT_AND_OFFSET.kicad_sch (KiCad schematic)
At the start: 6 parts, among them U1001 LMV321

Commit message: SUKU layout and hwcfg fixed
Other:
- note added: "[Simulation Link]"
Changed lines of the file:
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@@
 	(generator_version "10.0")
 	(paper "A4")
+	(text "[Simulation Link]"
+		(exclude_from_sim no)
+		(at 78.74 48.26 0)
+		(effects
+			(font
+				(size 1.27 1.27)
+				(thickness 0.254)
+				(bold yes)
+			)
+			(href "https://www.falstad.com/circuit/circuitjs.html?ctz=DwYwlgTgBAZgvAIgIwKgFwM6IAwDpsEECsqYIiSeATAVQOx0DM2AHFQGwCcndqIARoiLZUAB0EIALI1QA3CENQBbTEICmAWiQoAfACgoUYNAAeiDZJZQknKlEvXbqeAhFQFCIpREB6fYeAAQygzZHZsazp2KGZJSPZnRE5lQMRGXBkoJTAcVABzVORCAgQ-AyNTCnCoTmikavq3FzcPbxKygIB3EKqImzsHfsTXUv8KnrC+hur6KmGWimF2seA8icaoWesZlhZ50fLgACV16trtiPZJYfrUTuaUk1k0jIOuicHbeytb2FyOozdUKDaI0H4JP4jAHGCZg7YxbBxX4PdxCbxvCpAtKI+GxeL7HSxAA09QA3MSkFFgD4IJ0VrSJnjKdFJAR8ZCRITESSoqTWdgeexqbSVidQhYfl8NOchpDfvcKM4POFHs9kLgUFB+GBAlgEFRcOwSNCAPZQNQAOwocygGFEiCuwxMmXtIzGAVEUDVbgw5E8GI9XrSqF9OHw2CQRHYVGNKx8JpWZstFE1dod10hzrEivdRk93pDftj5UDasyodc4YIPCN0eLAXj+mp4Ag+iAA")
+		)
+	)
 	(junction
 		(at 111.76 73.66)
