File: Electrical/Design/PCBA-BU16/GRID.kicad_sch (KiCad schematic)
At the start: 9 parts, among them J501 Conn_01x04, J502 Conn_01x04, J503 Conn_01x04, J504 Conn_01x04, J505 Conn_01x04, J506 Conn_01x04, J507 Conn_01x04, J508 Conn_01x04, M501 Conn_01x08

Commit message: SUKU annotation checker added, wired into CI; BU16/EF44 reannotated
check_annotation.py verifies a schematic sheet instance's reference
designators against this repo's actual page-number-driven annotation
strategy (KiCad's "First free after sheet number X 100"), without
invoking KiCad — there's no headless reannotate to diff against, since
kicad-cli has no `sch annotate` and eeschema has no scripting console.
A sheet instance's page number gives it an exclusive numbering block;
each reference prefix gets its own Y-then-X sorted counter within it.
Multiply-instantiated sheets (e.g. UI_ENC_FILTER placed 4x, or
INVERT_AND_OFFSET nested 8x inside each of UI_HALL_PREAMP's 2
placements) are matched and checked per instance via KiCad's own
hierarchical path chains, not per file.

A preflight, required before any per-symbol check, walks the sheet
hierarchy from the project root (following Sheetfile references, same
as KiCad) and enforces two invariants the KiCad GUI does not: every
sheet instance's page number must be globally unique, and page numbers
must be contiguous from 1 with no gaps. It also flags .kicad_sch files
present in a design folder but unreachable from the root as orphans.

Wired into CI as "annotation-check" / "annotation gate", same pattern
as the existing schematic-drift/design-rules gates: GitHub Actions
error annotations plus a job-summary table when GITHUB_ACTIONS=true.
generate-artifacts now depends on it too.

Preflight caught a real bug in BU16: UI_HALL_PREAMP is placed twice,
and both placements' 8 nested INVERT_AND_OFFSET instances had been
assigned the same page numbers (11-18 each, duplicated) instead of
each getting its own range — invisible in KiCad's hierarchy panel
without instance-aware tooling. Fixed by renumbering one branch to
10-17 and the other to 19-26, then reannotating every sheet in both
EF44 and BU16 to match; both now pass with zero mismatches.

Also removed 6 orphaned .kicad_sch files (leftover from EF44's fork
off BU16 replacin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
Parts:
- renumbered J501 to J401, J502 to J402, J503 to J403, J504 to J404, J505 to J405, J506 to J406, J507 to J407, J508 to J408, M501 to M401
Other:
- note removed: "500"
Changed lines of the file:
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@@
-		)
-	)
-	(text "500"
-		(exclude_from_sim no)
-		(at 246.38 35.56 0)
-		(effects
-			(font
-				(size 10.16 10.16)
-				(thickness 2.032)
-				(bold yes)
-			)
-			(justify left bottom)
 		)
 	)
@@
 		(in_pos_files yes)
 		(dnp yes)
-		(property "Reference" "J504"
+		(property "Reference" "J404"
 			(at 50.8 55.88 90)
 			(show_name no)
@@
 			(project "PCBA-BU16"
 				(path "/e5217a0c-7f55-4c30-adda-7f8d95709d1b/00000000-0000-0000-0000-00005d757c78/00000000-0000-0000-0000-00005d85c9fc"
-					(reference "J504")
+					(reference "J404")
 					(unit 1)
 				)
@@
 		(in_pos_files yes)
 		(dnp yes)
-		(property "Reference" "J506"
+		(property "Reference" "J406"
 			(at 50.8 78.74 90)
 			(show_name no)
@@
 			(project "PCBA-BU16"
 				(path "/e5217a0c-7f55-4c30-adda-7f8d95709d1b/00000000-0000-0000-0000-00005d757c78/00000000-0000-0000-0000-00005d85c9fc"
-					(reference "J506")
+					(reference "J406")
 					(unit 1)
 				)
@@
 		(in_pos_files yes)
 		(dnp no)
-		(property "Reference" "#PWR0505"
+		(property "Reference" "#PWR0405"
 			(at 41.91 55.88 0)
 			(hide yes)
@@
 			(project "PCBA-BU16"
 				(path "/e5217a0c-7f55-4c30-adda-7f8d95709d1b/00000000-0000-0000-0000-00005d757c78/00000000-0000-0000-0000-00005d85c9fc"
-					(reference "#PWR0505")
+					(reference "#PWR0405")
 					(unit 1)
 				)
@@
 		(in_pos_files yes)
 		(dnp no)
-		(property "Reference" "#PWR0507"
+		(property "Reference" "#PWR0407"
 			(at 31.75 73.66 0)
 			(hide yes)
@@
 			(project "PCBA-BU16"
 				(path "/e5217a0c-7f55-4c30-adda-7f8d95709d1b/00000000-0000-0000-0000-00005d757c78/00000000-0000-0000-0000-00005d85c9fc"
-					(reference "#PWR0507")
+					(reference "#PWR0407")
 					(unit 1)
 				)
@@
 		(in_pos_files yes)
 		(dnp no)
-		(property "Reference" "#PWR0509"
+		(property "Reference" "#PWR0409"
 			(at 31.75 78.74 0)
 			(hide yes)
@@
 			(project "PCBA-BU16"
 				(path "/e5217a0c-7f55-4c30-adda-7f8d95709d1b/00000000-0000-0000-0000-00005d757c78/00000000-0000-0000-0000-00005d85c9fc"
-					(reference "#PWR0509")
+					(reference "#PWR0409")
 					(unit 1)
 				)
@@
 		(in_pos_files yes)
 		(dnp no)
-		(property "Reference" "#PWR0511"
+		(property "Reference" "#PWR0411"
 			(at 41.91 96.52 0)
 			(hide yes)
@@
 			(project "PCBA-BU16"
 				(path "/e5217a0c-7f55-4c30-adda-7f8d95709d1b/00000000-0000-0000-0000-00005d757c78/00000000-0000-0000-0000-00005d85c9fc"
-					(reference "#PWR0511")
+					(reference "#PWR0411")
 					(unit 1)
 				)
@@
 		(in_pos_files yes)
 		(dnp yes)
-		(property "Reference" "J502"
+		(property "Reference" "J402"
 			(at 96.52 50.8 90)
 			(show_name no)
@@
 			(project "PCBA-BU16"
 				(path "/e5217a0c-7f55-4c30-adda-7f8d95709d1b/00000000-0000-0000-0000-00005d757c78/00000000-0000-0000-0000-00005d85c9fc"
-					(reference "J502")
+					(reference "J402")
 					(unit 1)
 				)
@@
 		(in_pos_files yes)
 		(dnp yes)
-		(property "Reference" "J501"
+		(property "Reference" "J401"
 			(at 73.66 50.8 90)
 			(show_name no)
@@
 			(project "PCBA-BU16"
 				(path "/e5217a0c-7f55-4c30-adda-7f8d95709d1b/00000000-0000-0000-0000-00005d757c78/00000000-0000-0000-0000-00005d85c9fc"
-					(reference "J501")
+					(reference "J401")
 					(unit 1)
 				)
@@
 		(in_pos_files yes)
 		(dnp yes)
-		(property "Reference" "J505"
+		(property "Reference" "J405"
 			(at 101.6 96.52 90)
 			(show_name no)
@@
 			(project "PCBA-BU16"
 				(path "/e5217a0c-7f55-4c30-adda-7f8d95709d1b/00000000-0000-0000-0000-00005d757c78/00000000-0000-0000-0000-00005d85c9fc"
-					(reference "J505")
+					(reference "J405")
 					(unit 1)
 				)
@@
 		(in_pos_files yes)
 		(dnp yes)
-		(property "Reference" "J503"
+		(property "Reference" "J403"
 			(at 101.6 73.66 90)
 			(show_name no)
@@
 			(project "PCBA-BU16"
 				(path "/e5217a0c-7f55-4c30-adda-7f8d95709d1b/00000000-0000-0000-0000-00005d757c78/00000000-0000-0000-0000-00005d85c9fc"
-					(reference "J503")
+					(reference "J403")
 					(unit 1)
 				)
@@
 		(in_pos_files yes)
 		(dnp yes)
-		(property "Reference" "J507"
+		(property "Reference" "J407"
 			(at 55.88 101.6 90)
 			(show_name no)
@@
 			(project "PCBA-BU16"
 				(path "/e5217a0c-7f55-4c30-adda-7f8d95709d1b/00000000-0000-0000-0000-00005d757c78/00000000-0000-0000-0000-00005d85c9fc"
-					(reference "J507")
+					(reference "J407")
 					(unit 1)
 				)
@@
 		(in_pos_files yes)
 		(dnp yes)
-		(property "Reference" "J508"
+		(property "Reference" "J408"
 			(at 78.74 101.6 90)
 			(show_name no)
@@
 			(project "PCBA-BU16"
 				(path "/e5217a0c-7f55-4c30-adda-7f8d95709d1b/00000000-0000-0000-0000-00005d757c78/00000000-0000-0000-0000-00005d85c9fc"
-					(reference "J508")
+					(reference "J408")
 					(unit 1)
 				)
@@
 		(in_pos_files yes)
 		(dnp yes)
-		(property "Reference" "M501"
+		(property "Reference" "M401"
 			(at 180.34 73.66 90)
 			(show_name no)
@@
 			(project "PCBA-BU16"
 				(path "/e5217a0c-7f55-4c30-adda-7f8d95709d1b/00000000-0000-0000-0000-00005d757c78/00000000-0000-0000-0000-00005d85c9fc"
-					(reference "M501")
+					(reference "M401")
 					(unit 1)
 				)
@@
 		(in_pos_files yes)
 		(dnp no)
-		(property "Reference" "#PWR0516"
+		(property "Reference" "#PWR0416"
 			(at 96.52 110.49 0)
 			(hide yes)
@@
 			(project "PCBA-BU16"
 				(path "/e5217a0c-7f55-4c30-adda-7f8d95709d1b/00000000-0000-0000-0000-00005d757c78/00000000-0000-0000-0000-00005d85c9fc"
-					(reference "#PWR0516")
+					(reference "#PWR0416")
 					(unit 1)
 				)
@@
 		(in_pos_files yes)
 		(dnp no)
-		(property "Reference" "#PWR0506"
+		(property "Reference" "#PWR0406"
 			(at 110.49 55.88 0)
 			(hide yes)
@@
 			(project "PCBA-BU16"
 				(path "/e5217a0c-7f55-4c30-adda-7f8d95709d1b/00000000-0000-0000-0000-00005d757c78/00000000-0000-0000-0000-00005d85c9fc"
-					(reference "#PWR0506")
+					(reference "#PWR0406")
 					(unit 1)
 				)
@@
 		(in_pos_files yes)
 		(dnp no)
-		(property "Reference" "#PWR0512"
+		(property "Reference" "#PWR0412"
 			(at 110.49 96.52 0)
 			(hide yes)
@@
 			(project "PCBA-BU16"
 				(path "/e5217a0c-7f55-4c30-adda-7f8d95709d1b/00000000-0000-0000-0000-00005d757c78/00000000-0000-0000-0000-00005d85c9fc"
-					(reference "#PWR0512")
+					(reference "#PWR0412")
 					(unit 1)
 				)
@@
 		(in_pos_files yes)
 		(dnp no)
-		(property "Reference" "#PWR0504"
+		(property "Reference" "#PWR0404"
 			(at 96.52 41.91 0)
 			(hide yes)
@@
 			(project "PCBA-BU16"
 				(path "/e5217a0c-7f55-4c30-adda-7f8d95709d1b/00000000-0000-0000-0000-00005d757c78/00000000-0000-0000-0000-00005d85c9fc"
-					(reference "#PWR0504")
+					(reference "#PWR0404")
 					(unit 1)
 				)
@@
 		(in_pos_files yes)
 		(dnp no)
-		(property "Reference" "#PWR0510"
+		(property "Reference" "#PWR0410"
 			(at 120.65 78.74 0)
 			(hide yes)
@@
 			(project "PCBA-BU16"
 				(path "/e5217a0c-7f55-4c30-adda-7f8d95709d1b/00000000-0000-0000-0000-00005d757c78/00000000-0000-0000-0000-00005d85c9fc"
-					(reference "#PWR0510")
+					(reference "#PWR0410")
 					(unit 1)
 				)
@@
 		(in_pos_files yes)
 		(dnp no)
-		(property "Reference" "#PWR0503"
+		(property "Reference" "#PWR0403"
 			(at 78.74 31.75 0)
 			(hide yes)
@@
 			(project "PCBA-BU16"
 				(path "/e5217a0c-7f55-4c30-adda-7f8d95709d1b/00000000-0000-0000-0000-00005d757c78/00000000-0000-0000-0000-00005d85c9fc"
-					(reference "#PWR0503")
+					(reference "#PWR0403")
 					(unit 1)
 				)
@@
 		(in_pos_files yes)
 		(dnp no)
-		(property "Reference" "#PWR0502"
+		(property "Reference" "#PWR0402"
 			(at 73.66 31.75 0)
 			(hide yes)
@@
 			(project "PCBA-BU16"
 				(path "/e5217a0c-7f55-4c30-adda-7f8d95709d1b/00000000-0000-0000-0000-00005d757c78/00000000-0000-0000-0000-00005d85c9fc"
-					(reference "#PWR0502")
+					(reference "#PWR0402")
 					(unit 1)
 				)
@@
 		(in_pos_files yes)
 		(dnp no)
-		(property "Reference" "#PWR0514"
+		(property "Reference" "#PWR0414"
 			(at 73.66 120.65 0)
 			(hide yes)
@@
 			(project "PCBA-BU16"
 				(path "/e5217a0c-7f55-4c30-adda-7f8d95709d1b/00000000-0000-0000-0000-00005d757c78/00000000-0000-0000-0000-00005d85c9fc"
-					(reference "#PWR0514")
+					(reference "#PWR0414")
 					(unit 1)
 				)
@@
 		(in_pos_files yes)
 		(dnp no)
-		(property "Reference" "#PWR0501"
+		(property "Reference" "#PWR0401"
 			(at 55.88 41.91 0)
 			(hide yes)
@@
 			(project "PCBA-BU16"
 				(path "/e5217a0c-7f55-4c30-adda-7f8d95709d1b/00000000-0000-0000-0000-00005d757c78/00000000-0000-0000-0000-00005d85c9fc"
-					(reference "#PWR0501")
+					(reference "#PWR0401")
 					(unit 1)
 				)
@@
 		(in_pos_files yes)
 		(dnp no)
-		(property "Reference" "#PWR0515"
+		(property "Reference" "#PWR0415"
 			(at 78.74 120.65 0)
 			(hide yes)
@@
 			(project "PCBA-BU16"
 				(path "/e5217a0c-7f55-4c30-adda-7f8d95709d1b/00000000-0000-0000-0000-00005d757c78/00000000-0000-0000-0000-00005d85c9fc"
-					(reference "#PWR0515")
+					(reference "#PWR0415")
 					(unit 1)
 				)
@@
 		(in_pos_files yes)
 		(dnp no)
-		(property "Reference" "#PWR0508"
+		(property "Reference" "#PWR0408"
 			(at 120.65 73.66 0)
 			(hide yes)
@@
 			(project "PCBA-BU16"
 				(path "/e5217a0c-7f55-4c30-adda-7f8d95709d1b/00000000-0000-0000-0000-00005d757c78/00000000-0000-0000-0000-00005d85c9fc"
-					(reference "#PWR0508")
+					(reference "#PWR0408")
 					(unit 1)
 				)
@@
 		(in_pos_files yes)
 		(dnp no)
-		(property "Reference" "#PWR0513"
+		(property "Reference" "#PWR0413"
 			(at 55.88 110.49 0)
 			(hide yes)
@@
 			(project "PCBA-BU16"
 				(path "/e5217a0c-7f55-4c30-adda-7f8d95709d1b/00000000-0000-0000-0000-00005d757c78/00000000-0000-0000-0000-00005d85c9fc"
-					(reference "#PWR0513")
-					(unit 1)
-				)
+					(reference "#PWR0413")
+					(unit 1)
+				)
