File: Electrical/Design/PCBA-EF44/MCU.kicad_sch (KiCad schematic)
At the start: 57 parts, among them J701 C5137195, J702 Conn_02x05_Odd_Even, J799 Conn_01x02, SW701 C255807, SW702 C2905169, SW703 C2905169, U703 RP2040, U704 ESP32-S3, U705 W25Q64JVSSIQ, Y701 40MHz

Commit message: SUKU rp2350 variant of ef44, base project created from bu16
Parts:
- removed C731, C732, C735, C736, C737, C738, C740, C741, C744, C745, C747, C749, C751, C752: 100n, suku_basics:CAP_0402, symbol suku_basics:CAP
- removed C733, C734, C746, C754: 1u, suku_basics:CAP_0402, symbol suku_basics:CAP
- removed C739: 3p9, suku_basics:CAP_0402, symbol suku_basics:CAP
- removed C742: 1p8, suku_basics:CAP_0402, symbol suku_basics:CAP
- removed C743: 10u, suku_basics:CAP_0402, symbol suku_basics:CAP
- removed C748, C750: 10p, suku_basics:CAP_0402, symbol suku_basics:CAP
- removed C753: 10n, suku_basics:CAP_0402, symbol suku_basics:CAP
- removed J701: C5137195, Connector_Coaxial:U.FL_Molex_MCRF_73412-0110_Vertical, symbol Connector:Conn_Coaxial
- removed J702: Conn_02x05_Odd_Even, Connector_PinHeader_1.27mm:PinHeader_2x05_P1.27mm_Vertical, symbol Connector_Generic:Conn_02x05_Odd_Even
- removed L701: 1n8, suku_basics:IND_0402, symbol suku_basics:INDUCTOR
- removed L702: GZ2012D601TF, suku_basics:FERRIT_0805, symbol suku_basics:FERRIT
- removed R733, R736: 1k, suku_basics:RES_0402, symbol suku_basics:RES
- removed R735: 5k1, suku_basics:RES_0402, symbol suku_basics:RES
- removed TP701, TP702, TP703, TP704, TP706, TP707, TP708, TP709: TestPoint, TestPoint:TestPoint_Pad_D1.0mm, symbol Connector:TestPoint
- removed TP705, TP710: TestPoint, TestPoint:TestPoint_Pad_1.0x1.0mm, symbol Connector:TestPoint
- removed U703: RP2040, suku_basics:RP2040_QFN-56-1EP_7x7mm_P0.4mm_EP3.2x3.2mm, symbol suku_basics:RP2040
- removed U704: ESP32-S3, suku_basics:QFN-56-1EP_7x7mm_P0.4mm_EP3.2x3.2mm, symbol suku_basics:ESP32-S3
- removed Y701: 40MHz, Crystal:Crystal_SMD_Abracon_ABM8G-4Pin_3.2x2.5mm, symbol suku_basics:ESP32_XTAL
- added C608, C609: 10p, suku_basics:CAP_0402, symbol suku_basics:CAP
- added C610, C614, C615: 4u7, suku_basics:CAP_0402, symbol suku_basics:CAP
- added C611, C612, C613, C616, C617, C618, C619, C620, C621, C622, C623, C624: 100n, suku_basics:CAP_0402, symbol suku_basics:CAP
- added D602: 1N5819WS, Diode_SMD:D_SOD-323, symbol suku_basics:SCHOTTKY
- added L601: GXTC252010-3R3-MT, Inductor_SMD:L_1008_2520Metric, symbol suku_basics:INDUCTOR
- added R606, R607, R608: 27R, suku_basics:RES_0402, symbol suku_basics:RES
- added R611, R702, R737: 1k, suku_basics:RES_0402, symbol suku_basics:RES
- added R616: 0R, suku_basics:RES_0402, symbol suku_basics:RES
- added TP601: TestPoint, TestPoint:TestPoint_Pad_D1.0mm, symbol Connector:TestPoint
- added U609: RP2350A, Package_DFN_QFN:QFN-60-1EP_7x7mm_P0.4mm_EP3.4x3.4mm, symbol MCU_RaspberryPi:RP2350A
- added Y601: 12MHz, Crystal:Crystal_SMD_Abracon_ABM8G-4Pin_3.2x2.5mm, symbol suku_basics:ESP32_XTAL
- R701: value 5k1 -> 10k
- R734: value 5k1 -> 100k
- U705: value W25Q64JVSSIQ -> GD25B64ESIGR
Connections:
- net ESP_BOOT0 is gone; now on net GND: SW703.2 (B)
- net RP_RUN is gone; now on net RESET: R729.2
- net +1V1: now also C611.1, C612.1, C613.1, C614.1, L601.2, U609.23 (DVDD), U609.39 (DVDD), U609.50 (VREG_FB), U609.6 (DVDD)
- net +3V3: now also C616.1, C617.1, C618.1, C619.1, C620.1, C622.1, C623.1, C624.1, R606.1, R616.1, U609.1 (IOVDD), U609.11 (IOVDD), U609.20 (IOVDD), U609.30 (IOVDD), U609.38 (IOVDD), U609.44 (ADC_AVDD), U609.45 (IOVDD), U609.53 (USB_OTP_VDD)
- net GND: now also SW702.2 (B), C608.2, C609.2, C610.2, C611.2, C612.2, C613.2, C614.2, C615.2, C616.2, C617.2, C618.2, C619.2, C620.2, C621.2, C622.2, C623.2, C624.2, U609.47 (VREG_PGND), U609.61 (GND), Y601.2, Y601.4; no longer SW702.1 (A), SW703.1 (A)
- net GRID_EAST_RX: now also U609.33 (GPIO21)
- net GRID_EAST_TX: now also U609.32 (GPIO20)
- net GRID_NORTH_RX: now also U609.10 (GPIO7)
- net GRID_NORTH_TX: now also U609.34 (GPIO22)
- net GRID_SOUTH_RX: now also U609.31 (GPIO19)
- net GRID_SOUTH_TX: now also U609.14 (GPIO10)
- net GRID_SYNC_1: now also U609.35 (GPIO23)
- net GRID_SYNC_2: now also U609.8 (GPIO5)
- net GRID_WEST_RX: now also U609.13 (GPIO9)
- net GRID_WEST_TX: now also U609.12 (GPIO8)
- net HWCFG_CLOCK: now also U609.4 (GPIO2)
- net HWCFG_SHIFT: now also U609.3 (GPIO1)
- net LED_DATA_OUT: now also U609.9 (GPIO6)
- net MAP_MODE: now also SW701.1 (A), SW703.1 (A), D602.1 (K), R702.2, U609.27 (GPIO16); no longer C757.1
- net RP_SWCLK: now also U609.24 (SWCLK)
- net RP_SWDIO: now also U609.25 (SWDIO)
- net SPICLK: now also U609.56 (QSPI_SCLK)
- net SPICS0: now also R737.2, U609.60 (~{QSPI_SS})
- net SPID: now also U609.57 (QSPI_SD0)
- net SPIHD: now also U609.55 (QSPI_SD3)
- net SPIQ: now also U609.59 (QSPI_SD1)
- net SPIWP: now also U609.58 (QSPI_SD2)
- net USB_DN: now also R608.1
- net USB_DP: now also R607.1
- net VDD_SPI: now also C621.1, R616.2, U609.54 (QSPI_IOVDD)
- net ESP_RESET renamed RESET
- net RESET: now also SW702.1 (A), U609.26 (RUN); no longer SW702.2 (B)
- new net: C757.1, R702.1
- new net: R611.1, U609.22 (XOUT)
- new net: C609.1, R611.2, Y601.3
- new net: L601.1, U609.48 (VREG_LX)
- new net: D602.2 (A), R737.1
- new net: C608.1, U609.21 (XIN), Y601.1
- new net: C610.1, R606.2, U609.46 (VREG_AVDD)
- new net: R608.2, U609.51 (USB_DM)
- new net: R607.2, U609.52 (USB_DP)
- new net +5V: C615.1, U609.49 (VREG_VIN)
- new net A0: U609.37 (GPIO25)
- new net A1: U609.36 (GPIO24)
- new net ADC0: U609.40 (GPIO26/ADC0)
- new net ADC1: U609.41 (GPIO27/ADC1)
- new net ADC2: U609.42 (GPIO28/ADC2)
- new net ADC3: U609.43 (GPIO29/ADC3)
- new net HWCFG_DATA_IN: U609.7 (GPIO4)
- new net HWCFG_DATA_OUT: U609.5 (GPIO3)
- new net SPICS1: TP601.1, U609.2 (GPIO0)
- no-connect marks 20 -> 7
Other:
- note removed: "1.8nH LQG15HS1N8S02D 3.9pF GJM1555C1H3R9WB01D 1.8pF GJM1555C1H1R8BB01D"
- note removed: "Internal Pull-up"
- note removed: "LCSC: TXM40M0004322HBCEO00T S3240000091040JY"
- note removed: "Programming Interface"
- note removed: "U.FL-R-SMT-1(80)"
- moved on the sheet: C758, R729, SW702, SW703

Commit message: SUKU ef44 layout done
Changed lines of the file:
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@@
 	(wire
 		(pts
-			(xy 322.58 203.2) (xy 332.74 203.2)
-		)
-		(stroke
-			(width 0)
-			(type default)
-		)
-	)
-	(wire
-		(pts
 			(xy 119.38 167.64) (xy 119.38 170.18)
 		)
@@
 	(wire
 		(pts
-			(xy 332.74 203.2) (xy 332.74 200.66)
-		)
-		(stroke
-			(width 0)
-			(type default)
-		)
-	)
-	(wire
-		(pts
 			(xy 182.88 71.12) (xy 182.88 93.98)
 		)
@@
 					(unit 1)
 				)
-			)
-		)
-	)
-	(symbol
-		(lib_id "suku_basics:VDD_SPI")
-		(at 332.74 200.66 0)
-		(unit 1)
-		(body_style 1)
-		(exclude_from_sim no)
-		(in_bom yes)
-		(on_board yes)
-		(in_pos_files yes)
-		(dnp no)
-		(property "Reference" "#PWR0668"
-			(at 332.74 204.47 0)
-			(hide yes)
-			(show_name no)
-			(do_not_autoplace no)
-			(effects
-				(font
-					(size 1.27 1.27)
-				)
-			)
-		)
-		(property "Value" "VDD_SPI"
-			(at 332.74 195.58 0)
-			(show_name no)
-			(do_not_autoplace no)
-			(effects
-				(font
-					(size 1.27 1.27)
-				)
-			)
-		)
-		(property "Footprint" ""
-			(at 332.74 200.66 0)
-			(hide yes)
-			(show_name no)
-			(do_not_autoplace no)
-			(effects
-				(font
-					(size 1.27 1.27)
-				)
-			)
-		)
-		(property "Datasheet" ""
-			(at 332.74 200.66 0)
-			(hide yes)
-			(show_name no)
-			(do_not_autoplace no)
-			(effects
-				(font
-					(size 1.27 1.27)
-				)
-			)
-		)
-		(property "Description" "Power symbol creates a global label with name \"+3V3_UI\""
-			(at 332.74 200.66 0)
-			(hide yes)
-			(show_name no)
-			(do_not_autoplace no)
-			(effects
-				(font
-					(size 1.27 1.27)
-				)
-			)
-		)
-		(pin "1"
-		)
-		(instances
-			(project "PCBA-EF44"
-				(path "/e5217a0c-7f55-4c30-adda-7f8d95709d1b/00000000-0000-0000-0000-00005d757c78"
-					(reference "#PWR0668")
-					(unit 1)
-				)

Commit message: SUKU DRC strict schematic parity, duplicate footprints removed
Parts:
- LOGO701: now not fitted
Changed lines of the file:
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@@
 		(on_board yes)
 		(in_pos_files yes)
-		(dnp no)
+		(dnp yes)
 		(fields_autoplaced yes)
 		(property "Reference" "LOGO701"
