File: Electrical/Design/PCBA-EF44/HWCFG.kicad_sch (KiCad schematic)
At the start: 2 parts, among them U801 74HC165

Commit message: SUKU ef44 initial layout done
Parts:
- added JP801: (NF), Jumper:SolderJumper-2_P1.3mm_Open_TrianglePad1.0x1.5mm, symbol suku_basics:JP_SolderJumper_2_Open
- added R801: 5k1, suku_basics:RES_0402, symbol suku_basics:RES
Connections:
- net +3V3: now also U801.13 (D2), U801.4 (D5), JP801.1 (A); no longer U801.11 (D0), U801.6 (D7)
- net GND: now also U801.11 (D0), U801.6 (D7), R801.2; no longer U801.10 (SI), U801.13 (D2), U801.3 (D4), U801.4 (D5)
- net HWCFG_DATA_IN renamed HWCFG_DATA
- new net: JP801.2 (B), R801.1, U801.3 (D4)
- new net DATA_IN: U801.10 (SI)
Other:
- note added: "OPEN IF NORMAL ENCODER CLOSED IF NO DETENT"

Commit message: SUKU ef44 layout done
Parts:
- JP801: value (NF) -> ND; now not fitted
Changed lines of the file:
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@@
 			)
 		)
-		(property "Description" ""
+		(property "Description" "Power symbol creates a global label with name \"+3V3\""
 			(at 121.92 86.36 0)
 			(hide yes)
@@
 			)
 		)
-		(property "Description" ""
+		(property "Description" "Power symbol creates a global label with name \"GND\" , ground"
 			(at 121.92 101.6 0)
 			(hide yes)
@@
 		(on_board yes)
 		(in_pos_files yes)
-		(dnp no)
+		(dnp yes)
 		(property "Reference" "JP801"
 			(at 47.4472 77.5716 90)
@@
 			)
 		)
-		(property "Value" "(NF)"
+		(property "Value" "ND"
 			(at 47.4472 79.883 90)
 			(show_name no)
@@
 			)
 		)
-		(property "Description" ""
+		(property "Description" "Power symbol creates a global label with name \"+3V3\""
 			(at 104.14 63.5 0)
 			(hide yes)
@@
 			)
 		)
-		(property "Description" ""
+		(property "Description" "Power symbol creates a global label with name \"GND\" , ground"
 			(at 104.14 114.3 0)
 			(hide yes)
@@
 			)
 		)
-		(property "Description" ""
+		(property "Description" "Power symbol creates a global label with name \"GND\" , ground"
 			(at 45.72 93.98 0)
 			(hide yes)
@@
 			)
 		)
-		(property "Description" ""
+		(property "Description" "Power symbol creates a global label with name \"+3V3\""
 			(at 45.72 73.66 0)
 			(hide yes)
