File: Electrical/Design/PCBA-EF44/HWCFG.kicad_sch (KiCad schematic)
At the start: 4 parts, among them U801 74HC165

Commit message: SUKU annotation checker added, wired into CI; BU16/EF44 reannotated
check_annotation.py verifies a schematic sheet instance's reference
designators against this repo's actual page-number-driven annotation
strategy (KiCad's "First free after sheet number X 100"), without
invoking KiCad — there's no headless reannotate to diff against, since
kicad-cli has no `sch annotate` and eeschema has no scripting console.
A sheet instance's page number gives it an exclusive numbering block;
each reference prefix gets its own Y-then-X sorted counter within it.
Multiply-instantiated sheets (e.g. UI_ENC_FILTER placed 4x, or
INVERT_AND_OFFSET nested 8x inside each of UI_HALL_PREAMP's 2
placements) are matched and checked per instance via KiCad's own
hierarchical path chains, not per file.

A preflight, required before any per-symbol check, walks the sheet
hierarchy from the project root (following Sheetfile references, same
as KiCad) and enforces two invariants the KiCad GUI does not: every
sheet instance's page number must be globally unique, and page numbers
must be contiguous from 1 with no gaps. It also flags .kicad_sch files
present in a design folder but unreachable from the root as orphans.

Wired into CI as "annotation-check" / "annotation gate", same pattern
as the existing schematic-drift/design-rules gates: GitHub Actions
error annotations plus a job-summary table when GITHUB_ACTIONS=true.
generate-artifacts now depends on it too.

Preflight caught a real bug in BU16: UI_HALL_PREAMP is placed twice,
and both placements' 8 nested INVERT_AND_OFFSET instances had been
assigned the same page numbers (11-18 each, duplicated) instead of
each getting its own range — invisible in KiCad's hierarchy panel
without instance-aware tooling. Fixed by renumbering one branch to
10-17 and the other to 19-26, then reannotating every sheet in both
EF44 and BU16 to match; both now pass with zero mismatches.

Also removed 6 orphaned .kicad_sch files (leftover from EF44's fork
off BU16 replacin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
Parts:
- renumbered C801 to C501, JP801 to JP501, R801 to R501, U801 to U501
Other:
- note removed: "800"
Changed lines of the file:
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@@
 	(generator_version "10.0")
 	(paper "A4")
-	(text "800"
-		(exclude_from_sim no)
-		(at 25.4 33.02 0)
-		(effects
-			(font
-				(size 10.16 10.16)
-				(thickness 2.032)
-				(bold yes)
-			)
-			(justify left bottom)
-		)
-	)
 	(text "Board Identification\n\nGrid firmware can identify the hardware and the board \nrevision thorugh a 3 wire serial interface using one \nor more shift register as read only memory. The content\nof the memory is defined by pulling the inputs high or\nlow through pcb traces or solderable configuration jumpers.\n\n4b'Model + 4b'Revision + nb'Reserved (Multiple shift registers)\n\nD0: MODEL (LSB)\nD1: MODEL\nD2: MODEL\nD3: MODEL (MSB)\nD4: REVISION (LSB)\nD5: REVISION\nD6: REVISION\nD7: REVISION (MSB)\n\n\n\nModel Codes (D3-D0):\n\nPo16 0000\nBo16 0001\nPBF4 0010\nEN16 0011\n...\n\nRevision Codes (D7-D4):\n\nRevA 0000\nRevB 0001\nRevC 0010\nRevD 0011\n...\n"
 		(exclude_from_sim no)
@@
 		(dnp no)
 		(fields_autoplaced yes)
-		(property "Reference" "#PWR0803"
+		(property "Reference" "#PWR0503"
 			(at 121.92 90.17 0)
 			(hide yes)
@@
 			(project "PCBA-EF44"
 				(path "/e5217a0c-7f55-4c30-adda-7f8d95709d1b/00000000-0000-0000-0000-00005dc2dc06"
-					(reference "#PWR0803")
+					(reference "#PWR0503")
 					(unit 1)
 				)
@@
 		(in_pos_files yes)
 		(dnp no)
-		(property "Reference" "U801"
+		(property "Reference" "U501"
 			(at 93.98 63.5 0)
 			(show_name no)
@@
 			(project "PCBA-EF44"
 				(path "/e5217a0c-7f55-4c30-adda-7f8d95709d1b/00000000-0000-0000-0000-00005dc2dc06"
-					(reference "U801")
+					(reference "U501")
 					(unit 1)
 				)
@@
 		(in_pos_files yes)
 		(dnp no)
-		(property "Reference" "C801"
+		(property "Reference" "C501"
 			(at 124.2568 92.8116 0)
 			(show_name no)
@@
 			(project "PCBA-EF44"
 				(path "/e5217a0c-7f55-4c30-adda-7f8d95709d1b/00000000-0000-0000-0000-00005dc2dc06"
-					(reference "C801")
+					(reference "C501")
 					(unit 1)
 				)
@@
 		(in_pos_files yes)
 		(dnp no)
-		(property "Reference" "#PWR0805"
+		(property "Reference" "#PWR0505"
 			(at 121.92 107.95 0)
 			(hide yes)
@@
 			(project "PCBA-EF44"
 				(path "/e5217a0c-7f55-4c30-adda-7f8d95709d1b/00000000-0000-0000-0000-00005dc2dc06"
-					(reference "#PWR0805")
+					(reference "#PWR0505")
 					(unit 1)
 				)
@@
 		(in_pos_files yes)
 		(dnp yes)
-		(property "Reference" "JP801"
+		(property "Reference" "JP501"
 			(at 47.4472 77.5716 90)
 			(show_name no)
@@
 			(project "PCBA-EF44"
 				(path "/e5217a0c-7f55-4c30-adda-7f8d95709d1b/00000000-0000-0000-0000-00005dc2dc06"
-					(reference "JP801")
+					(reference "JP501")
 					(unit 1)
 				)
@@
 		(dnp no)
 		(fields_autoplaced yes)
-		(property "Reference" "#PWR0801"
+		(property "Reference" "#PWR0501"
 			(at 104.14 67.31 0)
 			(hide yes)
@@
 			(project "PCBA-EF44"
 				(path "/e5217a0c-7f55-4c30-adda-7f8d95709d1b/00000000-0000-0000-0000-00005dc2dc06"
-					(reference "#PWR0801")
+					(reference "#PWR0501")
 					(unit 1)
 				)
@@
 		(in_pos_files yes)
 		(dnp no)
-		(property "Reference" "#PWR0806"
+		(property "Reference" "#PWR0506"
 			(at 104.14 120.65 0)
 			(hide yes)
@@
 			(project "PCBA-EF44"
 				(path "/e5217a0c-7f55-4c30-adda-7f8d95709d1b/00000000-0000-0000-0000-00005dc2dc06"
-					(reference "#PWR0806")
+					(reference "#PWR0506")
 					(unit 1)
 				)
@@
 		(in_pos_files yes)
 		(dnp no)
-		(property "Reference" "#PWR0804"
+		(property "Reference" "#PWR0504"
 			(at 45.72 100.33 0)
 			(hide yes)
@@
 			(project "PCBA-EF44"
 				(path "/e5217a0c-7f55-4c30-adda-7f8d95709d1b/00000000-0000-0000-0000-00005dc2dc06"
-					(reference "#PWR0804")
+					(reference "#PWR0504")
 					(unit 1)
 				)
@@
 		(dnp no)
 		(fields_autoplaced yes)
-		(property "Reference" "#PWR0802"
+		(property "Reference" "#PWR0502"
 			(at 45.72 77.47 0)
 			(hide yes)
@@
 			(project "PCBA-EF44"
 				(path "/e5217a0c-7f55-4c30-adda-7f8d95709d1b/00000000-0000-0000-0000-00005dc2dc06"
-					(reference "#PWR0802")
+					(reference "#PWR0502")
 					(unit 1)
 				)
@@
 		(in_pos_files yes)
 		(dnp no)
-		(property "Reference" "R801"
+		(property "Reference" "R501"
 			(at 47.2186 87.7316 0)
 			(show_name no)
@@
 			(project "PCBA-EF44"
 				(path "/e5217a0c-7f55-4c30-adda-7f8d95709d1b/00000000-0000-0000-0000-00005dc2dc06"
-					(reference "R801")
+					(reference "R501")
 					(unit 1)
 				)
