File: Electrical/Design/FP-PBF4-DJ/FP-PBF4-DJ.kicad_pcb (KiCad board)
At the start: 2 copper layers, 105.6 x 105.6 mm, 22 parts

Commit message: SUKU jlcjlcjlc text removed from desings
Other:
- board text added: "${PROJECTNAME} ${HASH} ${DATE}"
- board text removed: "JLCJLCJLCJLC ${PROJECTNAME} ${HASH} ${DATE}"
Changed lines of the file:
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@@
 		)
 	)
-	(gr_text "JLCJLCJLCJLC\n${PROJECTNAME}\n${HASH}\n${DATE}"
+	(gr_text "${PROJECTNAME}\n${HASH}\n${DATE}"
 		(at 100 100 0)
 		(layer "B.SilkS")
