File: Electrical/Design/FP-VSN1-L/FP-VSN1-L.kicad_pcb (KiCad board)
At the start: 2 copper layers, 105.6 x 105.6 mm, 17 parts

Commit message: SUKU jlcjlcjlc text removed from desings
Other:
- board text added: "${PROJECTNAME} ${HASH} ${DATE}"
- board text removed: "JLCJLCJLCJLC ${PROJECTNAME} ${HASH} ${DATE}"
Changed lines of the file:
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@@
 		)
 	)
-	(gr_text "JLCJLCJLCJLC\n${PROJECTNAME}\n${HASH}\n${DATE}"
+	(gr_text "${PROJECTNAME}\n${HASH}\n${DATE}"
 		(at 105 92.5 0)
 		(layer "B.SilkS")

Commit message: SUKU helper silkscreen tect added to FP... designs
Other:
- board text added: "${LAYER} layer is intentionally empty, no printing is required on this design!"
Changed lines of the file:
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@@
+		)
+	)
+	(gr_text "${LAYER} layer is intentionally empty, no printing is required on this design!"
+		(at 100 160 0)
+		(layer "F.SilkS")
+		(effects
+			(font
+				(size 1 1)
+				(thickness 0.15)
+			)
 		)
 	)
