File: Electrical/Design/PCBA-PO16/UI_LED.kicad_sch (KiCad schematic)
At the start: 32 parts

Commit message: SUKU po16 cloned from bu16, added to preflight
Parts:
- removed D901: WS2812C-2020, suku_basics:UI_WS2812C-2020, symbol suku_basics:UI_WS2812C-2020
- added D601: XL-0807RGBC-2812B-S, suku_basics:UI_XL-0807RGBC-2812B-S, symbol suku_basics:UI_XL-0807RGBC-2812B-S
- D602: renamed from D905; value WS2812C-2020 -> XL-0807RGBC-2812B-S; footprint suku_basics:UI_WS2812C-2020 -> suku_basics:UI_XL-0807RGBC-2812B-S; symbol suku_basics:UI_WS2812C-2020 -> suku_basics:UI_XL-0807RGBC-2812B-S
- D603: renamed from D909; value WS2812C-2020 -> XL-0807RGBC-2812B-S; footprint suku_basics:UI_WS2812C-2020 -> suku_basics:UI_XL-0807RGBC-2812B-S; symbol suku_basics:UI_WS2812C-2020 -> suku_basics:UI_XL-0807RGBC-2812B-S
- D604: renamed from D913; value WS2812C-2020 -> XL-0807RGBC-2812B-S; footprint suku_basics:UI_WS2812C-2020 -> suku_basics:UI_XL-0807RGBC-2812B-S; symbol suku_basics:UI_WS2812C-2020 -> suku_basics:UI_XL-0807RGBC-2812B-S
- D605: renamed from D902; value WS2812C-2020 -> XL-0807RGBC-2812B-S; footprint suku_basics:UI_WS2812C-2020 -> suku_basics:UI_XL-0807RGBC-2812B-S; symbol suku_basics:UI_WS2812C-2020 -> suku_basics:UI_XL-0807RGBC-2812B-S
- D606: renamed from D906; value WS2812C-2020 -> XL-0807RGBC-2812B-S; footprint suku_basics:UI_WS2812C-2020 -> suku_basics:UI_XL-0807RGBC-2812B-S; symbol suku_basics:UI_WS2812C-2020 -> suku_basics:UI_XL-0807RGBC-2812B-S
- D607: renamed from D910; value WS2812C-2020 -> XL-0807RGBC-2812B-S; footprint suku_basics:UI_WS2812C-2020 -> suku_basics:UI_XL-0807RGBC-2812B-S; symbol suku_basics:UI_WS2812C-2020 -> suku_basics:UI_XL-0807RGBC-2812B-S
- D608: renamed from D914; value WS2812C-2020 -> XL-0807RGBC-2812B-S; footprint suku_basics:UI_WS2812C-2020 -> suku_basics:UI_XL-0807RGBC-2812B-S; symbol suku_basics:UI_WS2812C-2020 -> suku_basics:UI_XL-0807RGBC-2812B-S
- D609: renamed from D903; value WS2812C-2020 -> XL-0807RGBC-2812B-S; footprint suku_basics:UI_WS2812C-2020 -> suku_basics:UI_XL-0807RGBC-2812B-S; symbol suku_basics:UI_WS2812C-2020 -> suku_basics:UI_XL-0807RGBC-2812B-S
- D610: renamed from D907; value WS2812C-2020 -> XL-0807RGBC-2812B-S; footprint suku_basics:UI_WS2812C-2020 -> suku_basics:UI_XL-0807RGBC-2812B-S; symbol suku_basics:UI_WS2812C-2020 -> suku_basics:UI_XL-0807RGBC-2812B-S
- D611: renamed from D911; value WS2812C-2020 -> XL-0807RGBC-2812B-S; footprint suku_basics:UI_WS2812C-2020 -> suku_basics:UI_XL-0807RGBC-2812B-S; symbol suku_basics:UI_WS2812C-2020 -> suku_basics:UI_XL-0807RGBC-2812B-S
- D612: renamed from D915; value WS2812C-2020 -> XL-0807RGBC-2812B-S; footprint suku_basics:UI_WS2812C-2020 -> suku_basics:UI_XL-0807RGBC-2812B-S; symbol suku_basics:UI_WS2812C-2020 -> suku_basics:UI_XL-0807RGBC-2812B-S
- D613: renamed from D904; value WS2812C-2020 -> XL-0807RGBC-2812B-S; footprint suku_basics:UI_WS2812C-2020 -> suku_basics:UI_XL-0807RGBC-2812B-S; symbol suku_basics:UI_WS2812C-2020 -> suku_basics:UI_XL-0807RGBC-2812B-S
- D614: renamed from D908; value WS2812C-2020 -> XL-0807RGBC-2812B-S; footprint suku_basics:UI_WS2812C-2020 -> suku_basics:UI_XL-0807RGBC-2812B-S; symbol suku_basics:UI_WS2812C-2020 -> suku_basics:UI_XL-0807RGBC-2812B-S
- D615: renamed from D912; value WS2812C-2020 -> XL-0807RGBC-2812B-S; footprint suku_basics:UI_WS2812C-2020 -> suku_basics:UI_XL-0807RGBC-2812B-S; symbol suku_basics:UI_WS2812C-2020 -> suku_basics:UI_XL-0807RGBC-2812B-S
- D616: renamed from D916; value WS2812C-2020 -> XL-0807RGBC-2812B-S; footprint suku_basics:UI_WS2812C-2020 -> suku_basics:UI_XL-0807RGBC-2812B-S; symbol suku_basics:UI_WS2812C-2020 -> suku_basics:UI_XL-0807RGBC-2812B-S
- renumbered C901 to C601, C905 to C602, C909 to C603, C913 to C604, C902 to C605, C906 to C606, C910 to C607, C914 to C608, C903 to C609, C907 to C610, C911 to C611, C915 to C612, C904 to C613, C908 to C614, C912 to C615, C916 to C616
Connections:
- net +5V: now also D601.4 (VDD)
- net GND: now also D601.2 (VSS)
- net LED_DATA_IN: now also D601.3 (DIN)
- net at D602.3 (DIN): now also D601.1 (DOUT)
Other:
- note removed: "900"
