File: Electrical/Design/PCBA-PO16/UI_MUX.kicad_sch (KiCad schematic)
At the start: 18 parts, among them U1001 74HC4051

Commit message: SUKU po16 cloned from bu16, added to preflight
Parts:
- removed U1001: 74HC4051, suku_basics:SOIC-16_74HC4051, symbol suku_basics:74HC4051
- added U2701: 4052, suku_basics:SOIC-16_74HC4051, symbol 4xxx:4052
- renumbered C1001 to C2701, C1005 to C2702, C1002 to C2703, C1006 to C2704, C1003 to C2705, C1007 to C2706, C1004 to C2707, C1008 to C2708, C1009 to C2709, R1001 to R2701, R1005 to R2702, R1002 to R2703, R1006 to R2704, R1003 to R2705, R1007 to R2706, R1004 to R2707, R1008 to R2708
Connections:
- net +3V3: now also U2701.16 (VDD)
- net ADDRESS_A: now also U2701.10 (A)
- net ADDRESS_B: now also U2701.9 (B)
- net GND: now also U2701.6 (Inh), U2701.7 (VEE), U2701.8 (VSS)
- net at C2701.1, R2701.1: now also U2701.12 (X0)
- net at C2702.1, R2702.1: now also U2701.14 (X1)
- net at C2703.1, R2703.1: now also U2701.15 (X2)
- net at C2704.1, R2704.1: now also U2701.11 (X3)
- net at C2705.1, R2705.1: now also U2701.1 (Y0)
- net at C2706.1, R2706.1: now also U2701.5 (Y1)
- net at C2707.1, R2707.1: now also U2701.2 (Y2)
- net at C2708.1, R2708.1: now also U2701.4 (Y3)
- new net OUT0: U2701.13 (X)
- new net OUT1: U2701.3 (Y)

Commit message: SUKU layout done
Parts:
- renumbered C2701 to C801, C2702 to C802, C2703 to C803, C2704 to C804, C2705 to C805, C2706 to C806, C2707 to C807, C2708 to C808, C2709 to C809, R2701 to R801, R2702 to R802, R2703 to R803, R2704 to R804, R2705 to R805, R2706 to R806, R2707 to R807, R2708 to R808, U2701 to U801
Other:
- note removed: "1000"
